Commit message: removed fakejoint controller

File: moveo_DRL/src/moveo_description/urdf/goalPoint.urdf (robot description, URDF)
Before this commit: robot demo_cube, 1 links, 0 joints
Links:
- link my_box: geometry visual sphere radius=0.05
