Commit message: alles broken

File: moveo_DRL/src/moveo_description/urdf/links_joints.xacro (robot description, xacro)
@@ -2,5 +2,5 @@
 <robot xmlns:xacro="http://www.ros.org/wiki/xacro">
 <!-- https://bitbucket.org/theconstructcore/my-robotic-manipulator/src/master/urdf/links_joints.xacro -->
-  <xacro:macro name="m_joint" params="name type axis_xyz origin_rpy origin_xyz parent child limit_e limit_l limit_u limit_v mimic_joint:='' mimic_multiplier:=1 mimic_offset:=0 ">
+  <xacro:macro name="m_joint" params="name type axis_xyz origin_rpy origin_xyz parent child limit_e limit_l limit_u limit_v mimic_joint:='' mimic_multiplier:=1 mimic_offset:=0  passive_joint:=''">
     <joint name="${name}" type="${type}">
       <axis xyz="${axis_xyz}" />
@@ -13,4 +13,5 @@
       </xacro:if>
     </joint>
+    <xacro:unless value ="${passive_joint == 'passive'}">
     <transmission name="trans_${name}">
       <type>hardware_interface/PositionJointInterface</type>
@@ -23,6 +24,7 @@
       </actuator>
     </transmission>
+    </xacro:unless>
   </xacro:macro>
-<xacro:macro name="m_joint_passive" params="name type axis_xyz origin_rpy origin_xyz parent child limit_e limit_l limit_u limit_v mimic_joint:='' mimic_multiplier:=1 mimic_offset:=0 ">
+<!-- <xacro:macro name="m_joint_p" params="name type axis_xyz origin_rpy origin_xyz parent child limit_e limit_l limit_u limit_v mimic_joint:='' mimic_multiplier:=1 mimic_offset:=0  passive_joint:=''">
     <joint name="${name}" type="${type}">
       <axis xyz="${axis_xyz}" />
@@ -35,5 +37,17 @@
       </xacro:if>
     </joint>
-  </xacro:macro>
+  </xacro:macro> -->
+<!-- <xacro:macro name="m_joint_passive" params="name type axis_xyz origin_rpy origin_xyz parent child limit_e limit_l limit_u limit_v mimic_joint:='' mimic_multiplier:=1 mimic_offset:=0 ">
+    <joint name="${name}" type="${type}">
+      <axis xyz="${axis_xyz}" />
+      <limit effort="${limit_e}" lower="${limit_l}" upper="${limit_u}" velocity="${limit_v}" />
+      <origin rpy="${origin_rpy}" xyz="${origin_xyz}" />
+      <parent link="${parent}" />
+      <child link="${child}" />
+      <xacro:if value ="${mimic_joint !=''}">
+      <mimic joint="${mimic_joint}" multiplier="${mimic_multiplier}" offset="${mimic_offset}" />
+      </xacro:if>
+    </joint>
+  </xacro:macro> -->
 <xacro:macro name="m_joint_fixed" params="name origin_rpy origin_xyz parent child ">
     <joint name="${name}" type="fixed">
@@ -66,4 +80,21 @@
       </visual>
     </link>
+  </xacro:macro>
+  <xacro:macro name="mimic_joint_plugin_gazebo" params="name_prefix parent_joint mimic_joint has_pid:=false multiplier:=1.0 offset:=0 sensitiveness:=0.0 max_effort:=1.0 robot_namespace:=''">
+    <gazebo>
+      <plugin name="MimicJointPlugin" filename="libroboticsgroup_upatras_gazebo_mimic_joint_plugin.so">
+        <joint>${parent_joint}</joint>
+        <mimicJoint>${mimic_joint}</mimicJoint>
+        <xacro:if value="${has_pid}">
+        </xacro:if>
+        <multiplier>${multiplier}</multiplier>
+        <offset>${offset}</offset>
+        <sensitiveness>${sensitiveness}</sensitiveness>
+        <maxEffort>${max_effort}</maxEffort>
+        <xacro:unless value="${robot_namespace == ''}">
+          <robotNamespace>${robot_namespace}</robotNamespace>
+        </xacro:unless>
+      </plugin>
+    </gazebo>
   </xacro:macro>
 <!--

File: moveo_DRL/src/moveo_description/urdf/moveo.urdf.xacro (robot description, xacro)
@@ -209,10 +209,10 @@
         mass="0.008"
         origin_xyz_inertia ="-0.005681 0.000349 0.021391"
-        ixx="0.003081"
-        ixy="-0.000006"
-        ixz="0.000535"
-        iyy="0.002997"
-        iyz="0.000033"
-        izz="0.000457"
+        ixx="0.000003081"
+        ixy="-0.000000006"
+        ixz="0.000000535"
+        iyy="0.000002997"
+        iyz="0.000000033"
+        izz="0.000000457"
     />
     <xacro:m_joint name= "Tip_Gripper_Servo_Joint"
@@ -227,9 +227,13 @@
         limit_v="5"
         limit_e="5"
+        passive_joint="passive"
         mimic_joint="Gripper_Servo_Gear_Joint"
-        mimic_multiplier="1"
-        mimic_offset="0"
-    />
-    <xacro:m_link_mesh name="Gripper_Idol_Gear"
+        mimic_multiplier="-1"
+        mimic_offset="0"
+            />
+      <xacro:mimic_joint_plugin_gazebo name_prefix="Tip_Gripper_Servo_Joint"
+        parent_joint= "Gripper_Servo_Gear_Joint" mimic_joint="Tip_Gripper_Servo_Joint"
+        has_pid="false" multiplier="-1.0" max_effort="10000.0" />
+  <xacro:m_link_mesh name="Gripper_Idol_Gear"
         origin_xyz="0 0 0"
         origin_rpy="0 0 0"
@@ -245,5 +249,5 @@
         izz="0.112495"
     />
-       <xacro:m_joint name= "Gripper_Idol_Gear_Joint"
+        <xacro:m_joint name= "Gripper_Idol_Gear_Joint"
         type="revolute"
         origin_xyz= "-0.014 0 0.024"
@@ -252,10 +256,17 @@
         parent="Endeffector_Base"
         child="Gripper_Idol_Gear"
-        limit_l="0"
-        limit_u="0"
-        limit_v="5"
-        limit_e="5"
-    />
-     <xacro:m_link_mesh name="Tip_Gripper_Idol"
+        limit_l="-1.5707"
+        limit_u="1.5707"
+        limit_v="5"
+        limit_e="5"
+         mimic_joint="Gripper_Servo_Gear_Joint"
+        mimic_multiplier="-1"
+        mimic_offset="0"
+        passive_joint="passive"
+    />
+      <xacro:mimic_joint_plugin_gazebo name_prefix="Gripper_Idol_Gear_Joint"
+        parent_joint="Gripper_Servo_Gear_Joint" mimic_joint="Gripper_Idol_Gear_Joint"
+        has_pid="false" multiplier="-1.0" max_effort="10000.0" />
+      <xacro:m_link_mesh name="Tip_Gripper_Idol"
         origin_xyz="0 0 0"
         origin_rpy="0 0 0"
@@ -271,5 +282,5 @@
         izz="0.000457"
     />
-   <xacro:m_joint name= "Tip_Gripper_Idol_Joint"
+  <xacro:m_joint name= "Tip_Gripper_Idol_Joint"
         type="revolute"
         origin_xyz="0 0 0.04"
@@ -278,13 +289,17 @@
         parent="Gripper_Idol_Gear"
         child="Tip_Gripper_Idol"
-        limit_l="-1.5"
-        limit_u="0"
-        limit_v="5"
-        limit_e="5"
-        mimic_joint="Gripper_Idol_Gear_Joint"
-        mimic_multiplier="-1"
-        mimic_offset="0"
-    />
-     <xacro:m_link_mesh name="Pivot_Arm_Gripper_Servo"
+        limit_l="-1.5707"
+        limit_u="1.5707"
+        limit_v="5"
+        limit_e="5"
+        mimic_joint="Gripper_Servo_Gear_Joint"
+        mimic_multiplier="1"
+        mimic_offset="0"
+        passive_joint="passive"
+    />
+   <xacro:mimic_joint_plugin_gazebo name_prefix="Tip_Gripper_Idol_Joint"
+    parent_joint="Gripper_Servo_Gear_Joint" mimic_joint="Tip_Gripper_Idol_Joint"
+    has_pid="false" multiplier="1.0" max_effort="10000.0" />
+   <!-- <xacro:m_link_mesh name="Pivot_Arm_Gripper_Servo"
         origin_xyz="0 0 0"
         origin_rpy="0 0 0"
@@ -314,6 +329,11 @@
         mimic_multiplier="1"
         mimic_offset="0"
-    />
-     <xacro:m_link_mesh name="Pivot_Arm_Gripper_Idol"
+        passive_joint="passive"
+    />
+     <xacro:mimic_joint_plugin_gazebo name_prefix="Mimic"
+    parent_joint="Gripper_Servo_Gear_Joint" mimic_joint="Pivot_Arm_Gripper_Servo_Joint"
+    has_pid="false" multiplier="1.0" max_effort="10000.0" />
+     -->
+      <xacro:m_link_mesh name="Pivot_Arm_Gripper_Idol"
         origin_xyz="0 0 0"
         origin_rpy="0 0 0"
@@ -340,10 +360,15 @@
         limit_v="5"
         limit_e="5"
-        mimic_joint="Gripper_Idol_Gear_Joint"
-        mimic_multiplier="1"
-        mimic_offset="0"
-    />
+        mimic_joint="Gripper_Servo_Gear_Joint"
+        mimic_multiplier="-1"
+        mimic_offset="0"
+        passive_joint="passive"
+    />
+     <xacro:mimic_joint_plugin_gazebo name_prefix="Mimic"
+    parent_joint="Gripper_Servo_Gear_Joint" mimic_joint="Pivot_Arm_Gripper_Idol_Joint"
+    has_pid="false" multiplier="-1.0" max_effort="10000.0" />
     <gazebo>
         <plugin name="gazebo_ros_control" filename="libgazebo_ros_control.so"/>
+       <!-- <plugin name="MimicJointPlugin" filename="libroboticsgroup_upatras_gazebo_mimic_joint_plugin.so"/>  -->
     </gazebo>
 </robot>

Commit message: added RealRobotControl as well as loading policies

File: moveo_DRL/src/moveo_description/urdf/links_joints.xacro (robot description, xacro)
@@ -62,5 +62,5 @@
         <mass value="${mass}" />
         <origin rpy="${origin_rpy_inertia}" xyz="${origin_xyz_inertia}" />
-        <inertia  ixx="${ixx}" ixy="${ixy}" ixz="${ixz}" iyy="${iyy}" iyz="${iyz}" izz="${izz}" />
+        <inertia  ixx="${0.01*ixx}" ixy="${0.01*ixy}" ixz="${0.01*ixz}" iyy="${0.01*iyy}" iyz="${0.01*iyz}" izz="${0.01*izz}" />
       </inertial>
       <collision>

File: moveo_DRL/src/moveo_description/urdf/moveo.urdf.xacro (robot description, xacro)
@@ -162,11 +162,11 @@
         meshfile_collision= "${path_to_meshes}/Base_Endeffektor.stl"
         mass="0.222"
-        origin_xyz_inertia ="-0.000548 0.000367 0.01865"
-        ixx="0.0009149"
-        ixy="0.00006"
-        ixz="0.000065"
-        iyy="0.010259"
-        iyz="-0.000101"
-        izz="0.005846"
+        origin_xyz_inertia ="0.002106 0.02106 0.022049"
+        ixx="0.028064"
+        ixy="-0.002005"
+        ixz="-0.000247"
+        iyy="0.017627"
+        iyz="-0.002423"
+        izz="0.028786"
     />
      <xacro:m_joint_fixed name= "Endeffector_Link_5_Joint"
@@ -181,12 +181,12 @@
         meshfile_visual= "${path_to_meshes}/Servo_Gear.stl"
         meshfile_collision= "${path_to_meshes}/Servo_Gear.stl"
-        mass="0.002453"
-        origin_xyz_inertia ="-0.000406 0 0.006451"
-        ixx="0.469425"
-        ixy="0"
-        ixz="-0.00957"
-        iyy="0.567572"
-        iyz="0"
-        izz="0.112495"
+        mass="0.002391"
+        origin_xyz_inertia ="0.000396 0 0.006595"
+        ixx="0.000466195"
+        ixy="0"
+        ixz="-0.0008252"
+        iyy="0.000564010"
+        iyz="0"
+        izz="0.000111803"
     />
    <xacro:m_joint name= "Gripper_Servo_Gear_Joint"
@@ -209,10 +209,10 @@
         mass="0.008"
         origin_xyz_inertia ="-0.005681 0.000349 0.021391"
-        ixx="0.000003081"
-        ixy="-0.000000006"
-        ixz="0.000000535"
-        iyy="0.000002997"
-        iyz="0.000000033"
-        izz="0.000000457"
+        ixx="0.003081"
+        ixy="-0.000006"
+        ixz="0.000535"
+        iyy="0.002997"
+        iyz="0.000033"
+        izz="0.000457"
     />
     <xacro:m_joint name= "Tip_Gripper_Servo_Joint"
@@ -241,11 +241,11 @@
         meshfile_collision= "${path_to_meshes}/Idol_Gear.stl"
         mass="0.002453"
-        origin_xyz_inertia ="-0.000406 0 0.006451"
-        ixx="0.469425"
-        ixy="0"
-        ixz="0.00957"
-        iyy="0.567572"
-        iyz="0"
-        izz="0.112495"
+        origin_xyz_inertia ="-0.000407 0 0.006453"
+        ixx="0.000469369"
+        ixy="0"
+        ixz="-0.000009589"
+        iyy="0.000567491"
+        iyz="0"
+        izz="0.00011247"
     />
         <xacro:m_joint name= "Gripper_Idol_Gear_Joint"
@@ -342,10 +342,10 @@
         mass="0.001638"
         origin_xyz_inertia ="0.005681  0.000349 0.021391"
-        ixx="0.303761"
+        ixx="0.000303761"
         ixy="0"
         ixz="0"
-        iyy="0.304662"
-        iyz="0"
-        izz="0.010301"
+        iyy="0.000304662"
+        iyz="0"
+        izz="0.000010301"
     />
     <xacro:m_joint name= "Pivot_Arm_Gripper_Idol_Joint"
